File: Kicad9_projects_folder/MY-ESP32/Battery_Voltage_Monitor_with_MOSFETS.kicad_sch (KiCad schematic)
At the start: 6 parts, among them Q3 N-MOSFET-ENH-2N7002, Q4 P-MOSFET-ENH-BSS84LT1G

Commit message: Second commit
Parts:
- renumbered R16 to R13, R17 to R14, R18 to R15, R19 to R16
Other:
- moved on the sheet: Q3, R13, R14, R15, R16
