File: Kicad9_projects_folder/MY-ESP32/Buck-Boost3.3V.kicad_sch (KiCad schematic)
At the start: 7 parts, among them U5 TPS63001DRCR

Commit message: Third commit
Connections:
- net Buck-Boost_EN is gone; now on net Buck-Boost_INPUT: U5.6 (EN)
Changed lines of the file:
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@@
+	)
+	(junction
+		(at 125.73 99.06)
+		(diameter 0)
+		(color 0 0 0 0)
 	)
 	(junction
@@
 	(wire
 		(pts
+			(xy 125.73 99.06) (xy 125.73 93.98)
+		)
+		(stroke
+			(width 0)
+			(type default)
+		)
+	)
+	(wire
+		(pts
 			(xy 140.97 72.39) (xy 128.27 72.39)
 		)
@@
 	(wire
 		(pts
-			(xy 129.54 99.06) (xy 129.54 144.78)
-		)
-		(stroke
-			(width 0)
-			(type default)
-		)
-	)
-	(wire
-		(pts
 			(xy 67.31 93.98) (xy 67.31 97.79)
 		)
@@
 	(wire
 		(pts
-			(xy 129.54 99.06) (xy 132.08 99.06)
-		)
-		(stroke
-			(width 0)
-			(type default)
-		)
-	)
-	(wire
-		(pts
 			(xy 168.91 107.95) (xy 168.91 106.68)
 		)
@@
 	(wire
 		(pts
-			(xy 125.73 106.68) (xy 125.73 93.98)
+			(xy 125.73 106.68) (xy 125.73 99.06)
 		)
 		(stroke
@@
 	(wire
 		(pts
-			(xy 129.54 144.78) (xy 124.46 144.78)
+			(xy 125.73 99.06) (xy 132.08 99.06)
 		)
 		(stroke
@@
 		(effects
 			(font
-				(size 1.27 1.27)
-			)
-			(justify right)
-		)
-	)
-	(hierarchical_label "Buck-Boost_EN"
-		(shape input)
-		(at 124.46 144.78 180)
-		(effects
-			(font

Commit message: Second commit
Parts:
- renumbered C15 to C11, C16 to C12, C17 to C13, C18 to C14, R20 to R17
Changed lines of the file:
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@@
 		(instances
 			(project "MY-ESP32"
-				(path "/d6d8d651-8dd4-45a4-bd17-f84a87bbb30c/7efd7115-3e45-40c0-b344-3c012cbc13c1"
+				(path "/d6d8d651-8dd4-45a4-bd17-f84a87bbb30c/bd1333f1-cd43-4d31-a242-4960306cc242"
 					(reference "#PWR051")
 					(unit 1)
@@
 		(instances
 			(project "MY-ESP32"
-				(path "/d6d8d651-8dd4-45a4-bd17-f84a87bbb30c/7efd7115-3e45-40c0-b344-3c012cbc13c1"
+				(path "/d6d8d651-8dd4-45a4-bd17-f84a87bbb30c/bd1333f1-cd43-4d31-a242-4960306cc242"
 					(reference "#PWR047")
 					(unit 1)
@@
 		(instances
 			(project "MY-ESP32"
-				(path "/d6d8d651-8dd4-45a4-bd17-f84a87bbb30c/7efd7115-3e45-40c0-b344-3c012cbc13c1"
+				(path "/d6d8d651-8dd4-45a4-bd17-f84a87bbb30c/bd1333f1-cd43-4d31-a242-4960306cc242"
 					(reference "#PWR048")
 					(unit 1)
@@
 		)
 		(instances
-			(project ""
-				(path "/d6d8d651-8dd4-45a4-bd17-f84a87bbb30c/7efd7115-3e45-40c0-b344-3c012cbc13c1"
+			(project "MY-ESP32"
+				(path "/d6d8d651-8dd4-45a4-bd17-f84a87bbb30c/bd1333f1-cd43-4d31-a242-4960306cc242"
 					(reference "U5")
 					(unit 1)
@@
 		(on_board yes)
 		(dnp no)
-		(property "Reference" "R20"
+		(property "Reference" "R17"
 			(at 231.394 100.33 90)
 			(effects
@@
 		)
 		(instances
-			(project ""
-				(path "/d6d8d651-8dd4-45a4-bd17-f84a87bbb30c/7efd7115-3e45-40c0-b344-3c012cbc13c1"
-					(reference "R20")
+			(project "MY-ESP32"
+				(path "/d6d8d651-8dd4-45a4-bd17-f84a87bbb30c/bd1333f1-cd43-4d31-a242-4960306cc242"
+					(reference "R17")
 					(unit 1)
 				)
@@
 		(on_board yes)
 		(dnp no)
-		(property "Reference" "C15"
+		(property "Reference" "C11"
 			(at 53.34 101.092 90)
 			(effects
@@
 		)
 		(instances
-			(project ""
-				(path "/d6d8d651-8dd4-45a4-bd17-f84a87bbb30c/7efd7115-3e45-40c0-b344-3c012cbc13c1"
-					(reference "C15")
+			(project "MY-ESP32"
+				(path "/d6d8d651-8dd4-45a4-bd17-f84a87bbb30c/bd1333f1-cd43-4d31-a242-4960306cc242"
+					(reference "C11")
 					(unit 1)
 				)
@@
 		(instances
 			(project "MY-ESP32"
-				(path "/d6d8d651-8dd4-45a4-bd17-f84a87bbb30c/7efd7115-3e45-40c0-b344-3c012cbc13c1"
+				(path "/d6d8d651-8dd4-45a4-bd17-f84a87bbb30c/bd1333f1-cd43-4d31-a242-4960306cc242"
 					(reference "#PWR050")
 					(unit 1)
@@
 		(on_board yes)
 		(dnp no)
-		(property "Reference" "C18"
+		(property "Reference" "C14"
 			(at 196.342 100.076 90)
 			(effects
@@
 		)
 		(instances
-			(project ""
-				(path "/d6d8d651-8dd4-45a4-bd17-f84a87bbb30c/7efd7115-3e45-40c0-b344-3c012cbc13c1"
-					(reference "C18")
+			(project "MY-ESP32"
+				(path "/d6d8d651-8dd4-45a4-bd17-f84a87bbb30c/bd1333f1-cd43-4d31-a242-4960306cc242"
+					(reference "C14")
 					(unit 1)
 				)
@@
 		(instances
 			(project "MY-ESP32"
-				(path "/d6d8d651-8dd4-45a4-bd17-f84a87bbb30c/7efd7115-3e45-40c0-b344-3c012cbc13c1"
+				(path "/d6d8d651-8dd4-45a4-bd17-f84a87bbb30c/bd1333f1-cd43-4d31-a242-4960306cc242"
 					(reference "#PWR052")
 					(unit 1)
@@
 		(on_board yes)
 		(dnp no)
-		(property "Reference" "C17"
+		(property "Reference" "C13"
 			(at 176.53 98.552 90)
 			(effects
@@
 		(instances
 			(project "MY-ESP32"
-				(path "/d6d8d651-8dd4-45a4-bd17-f84a87bbb30c/7efd7115-3e45-40c0-b344-3c012cbc13c1"
-					(reference "C17")
+				(path "/d6d8d651-8dd4-45a4-bd17-f84a87bbb30c/bd1333f1-cd43-4d31-a242-4960306cc242"
+					(reference "C13")
 					(unit 1)
 				)
@@
 		(instances
 			(project "MY-ESP32"
-				(path "/d6d8d651-8dd4-45a4-bd17-f84a87bbb30c/7efd7115-3e45-40c0-b344-3c012cbc13c1"
+				(path "/d6d8d651-8dd4-45a4-bd17-f84a87bbb30c/bd1333f1-cd43-4d31-a242-4960306cc242"
 					(reference "#PWR053")
 					(unit 1)
@@
 		)
 		(instances
-			(project ""
-				(path "/d6d8d651-8dd4-45a4-bd17-f84a87bbb30c/7efd7115-3e45-40c0-b344-3c012cbc13c1"
+			(project "MY-ESP32"
+				(path "/d6d8d651-8dd4-45a4-bd17-f84a87bbb30c/bd1333f1-cd43-4d31-a242-4960306cc242"
 					(reference "L_B-B1")
 					(unit 1)
@@
 		(on_board yes)
 		(dnp no)
-		(property "Reference" "C16"
+		(property "Reference" "C12"
 			(at 74.422 100.584 0)
 			(effects
@@
 		(instances
 			(project "MY-ESP32"
-				(path "/d6d8d651-8dd4-45a4-bd17-f84a87bbb30c/7efd7115-3e45-40c0-b344-3c012cbc13c1"
-					(reference "C16")
-					(unit 1)
-				)
+				(path "/d6d8d651-8dd4-45a4-bd17-f84a87bbb30c/bd1333f1-cd43-4d31-a242-4960306cc242"
+					(reference "C12")
+					(unit 1)
+				)
