File: Kicad9_projects_folder/MY-ESP32/MY-ESP32.kicad_pcb (KiCad board)
At the start: 4 copper layers, 97.3 x 90.9 mm, 99 parts, among them Q1 2N3904S-RTK/PS, Q2 2N3904S-RTK/PS, Q3 N-MOSFET-ENH-2N7002, Q4 P-MOSFET-ENH-BSS84LT1G, Q5 PMOSFET-DMP1045U-7, SW1 BOOT, SW2 RESET, U1 USBLC6-2SC6, U10 USB-C_Connector, U11 TPS3839G33DBZR, U2 Screw_Terminal_KF301_1x02, U3 CP2102N-Axx-xQFN28, U5 TPS63001DRCR, U7 LTC4121EUD#TRPBF

Commit message: Second commit
Parts:
- removed the ? at (140.7, 87.7)
- removed the ? at (142.1, 121.3)
- removed the ? at (139.8, 86.8)
- removed the ? at (138.8, 86.8)
- removed the ? at (140.7, 85.9)
- removed the ? at (137.9, 86.8)
- removed the ? at (143.3, 121.3)
- removed the ? at (137.0, 85.9)
- removed the ? at (137.9, 84.9)
- removed the ? at (137.9, 88.6)
- removed the ? at (138.9, 87.7)
- removed the ? at (139.8, 84.9)
- removed the ? at (138.9, 85.9)
- removed the ? at (139.8, 88.6)
- removed the ? at (137.0, 87.7)
- removed the ? at (142.7, 121.3)
- added ?: , , F.Cu at (39.7, 62.4)
- added ?: , , F.Cu at (59.6, 29.9)
- added ?: , , F.Cu at (57.8, 31.7)
- added ?: , , F.Cu at (44.2, 88.3)
- added ?: , , F.Cu at (43.1, 87.1)
- added ?: , , F.Cu at (63.8, 65.3)
- added ?: , , F.Cu at (61.5, 28.0)
- added ?: , , F.Cu at (43.1, 88.3)
- added ?: , , F.Cu at (59.6, 31.7)
- added ?: , , F.Cu at (40.7, 63.3)
- added ?: , , F.Cu at (64.4, 65.3)
- added ?: , , F.Cu at (61.5, 33.6)
- added ?: , , F.Cu at (44.2, 87.1)
- added ?: , , F.Cu at (63.4, 33.6)
- added ?: , , F.Cu at (59.6, 28.0)
- added ?: , , F.Cu at (61.5, 31.7)
- added ?: , , F.Cu at (63.4, 31.7)
- added ?: , , F.Cu at (65.0, 65.3)
- added ?: , , F.Cu at (40.7, 62.4)
- added ?: , , F.Cu at (59.6, 33.6)
- added ?: , , F.Cu at (63.4, 28.0)
- added ?: , , F.Cu at (39.7, 63.3)
- added ?: , , F.Cu at (63.4, 29.9)
- added ?: , , F.Cu at (57.8, 29.9)
- added ?: , , F.Cu at (57.8, 33.6)
- added ?: , , F.Cu at (57.8, 28.0)
- added ?: , , F.Cu at (61.5, 29.9)
- added R24: 7.5kΩ, My_Personal_Footprints_Library:0603WAF7501T5E, F.Cu at (100.5, 39.7)
- added R25: 7.5kΩ, My_Personal_Footprints_Library:0603WAF7501T5E, F.Cu at (100.6, 41.8)
- added R26: 7.5kΩ, My_Personal_Footprints_Library:0603WAF7501T5E, F.Cu at (103.2, 53.7)
- moved C2 96.2 mm to (73.6, 82.1)
- moved H10 96.2 mm to (117.3, 22.3)
- moved H13 96.2 mm to (117.3, 66.6)
- moved H6 96.2 mm to (113.5, 57.7)
- moved H8 96.2 mm to (100.7, 34.8)
- moved R23 96.2 mm to (103.3, 51.0)
- moved TP3 96.2 mm to (64.7, 51.9)
- moved C1 96.2 mm to (74.1, 91.1)
- moved C10 96.2 mm to (101.9, 46.5)
- moved C11 96.2 mm to (42.0, 69.0)
- moved C12 96.2 mm to (42.4, 66.4)
- moved C13 96.2 mm to (38.4, 65.6)
- moved C15 96.2 mm to (61.3, 64.4)
- moved C17 96.2 mm to (69.6, 64.4)
- moved C18 96.2 mm to (67.4, 64.4)
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Connections:
- CARD1 pad 1: unconnected-(CARD1-DAT2-Pad1) -> Net-(CARD1-DAT2)
- CARD1 pad 2: unconnected-(CARD1-CD/DAT3-Pad2) -> Net-(CARD1-CD/DAT3)
- CARD1 pad 8: unconnected-(CARD1-DAT1-Pad8) -> Net-(CARD1-DAT1)
Routing:
- net +3V3: track 267.4 -> 282.9 mm, vias 10 -> 13
- net GND: track 161.3 -> 152.1 mm, vias 29 -> 32
- net Net-(CARD1-DAT2): track 0.00 -> 7.53 mm
- net Net-(CARD1-CD/DAT3): track 0.00 -> 7.02 mm
- net Net-(CARD1-DAT1): track 0.00 -> 3.57 mm
- net D35: track 76.1 -> 79.5 mm
- net /Buck-Boost3.3V/Buck-Boost_EN: track 30.7 -> 27.9 mm
- net D26: track 50.9 -> 52.8 mm
- net D32: track 72.8 -> 74.5 mm
- net D23: track 54.7 -> 56.0 mm
- net EXT_5V: track 164.9 -> 164.0 mm
- net /Buck-Boost3.3V/Buck-Boost_INPUT: track 33.1 -> 32.3 mm
- net D22: track 51.7 -> 52.6 mm
- net D15: track 43.3 -> 42.5 mm
- net D5: track 41.2 -> 40.6 mm
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
Commit message: Third commit
Parts:
- removed the ? at (39.7, 62.4)
- removed the ? at (59.6, 29.9)
- removed the ? at (57.8, 31.7)
- removed the ? at (44.2, 88.3)
- removed the ? at (43.1, 87.1)
- removed the ? at (63.8, 65.3)
- removed the ? at (61.5, 28.0)
- removed the ? at (43.1, 88.3)
- removed the ? at (59.6, 31.7)
- removed the ? at (40.7, 63.3)
- removed the ? at (64.4, 65.3)
- removed the ? at (61.5, 33.6)
- removed the ? at (44.2, 87.1)
- removed the ? at (63.4, 33.6)
- removed the ? at (59.6, 28.0)
- removed the ? at (61.5, 31.7)
- removed the ? at (63.4, 31.7)
- removed the ? at (65.0, 65.3)
- removed the ? at (40.7, 62.4)
- removed the ? at (59.6, 33.6)
- removed the ? at (63.4, 28.0)
- removed the ? at (39.7, 63.3)
- removed the ? at (63.4, 29.9)
- removed the ? at (57.8, 29.9)
- removed the ? at (57.8, 33.6)
- removed the ? at (57.8, 28.0)
- removed the ? at (61.5, 29.9)
- removed U11: TPS3839G33DBZR, My_Personal_Footprints_Library:TPS3839G33DBZR
- added ?: , , F.Cu at (44.2, 87.1)
- added ?: , , F.Cu at (59.7, 33.6)
- added ?: , , F.Cu at (63.4, 31.7)
- added ?: , , F.Cu at (43.1, 87.1)
- added ?: , , F.Cu at (57.8, 33.6)
- added ?: , , F.Cu at (63.4, 28.0)
- added ?: , , F.Cu at (64.4, 65.3)
- added ?: , , F.Cu at (61.5, 29.9)
- added ?: , , F.Cu at (57.8, 29.9)
- added ?: , , F.Cu at (61.5, 28.0)
- added ?: , , F.Cu at (61.5, 33.6)
- added ?: , , F.Cu at (57.8, 31.7)
- added ?: , , F.Cu at (57.8, 28.0)
- added ?: , , F.Cu at (65.0, 65.3)
- added ?: , , F.Cu at (63.4, 29.9)
- added ?: , , F.Cu at (59.7, 28.0)
- added ?: , , F.Cu at (59.7, 31.7)
- added ?: , , F.Cu at (44.2, 88.3)
- added ?: , , F.Cu at (63.8, 65.3)
- added ?: , , F.Cu at (59.7, 29.9)
- added ?: , , F.Cu at (61.5, 31.7)
- added ?: , , F.Cu at (43.1, 88.3)
- added ?: , , F.Cu at (63.4, 33.6)
Connections:
- U5 pad 6: /Buck-Boost3.3V/Buck-Boost_EN -> /Buck-Boost3.3V/Buck-Boost_INPUT
Routing:
- net /Buck-Boost3.3V/Buck-Boost_EN: track 27.9 -> 0.00 mm
- net /Battery_Charger_LiFePO4_3.6V/Battery_Charger_OUTPUT: track 77.3 -> 59.7 mm
- net GND: track 152.1 -> 150.3 mm
- net /Buck-Boost3.3V/Buck-Boost_INPUT: track 32.3 -> 33.4 mm

Commit message: Second commit
Parts:
- removed the ? at (44.2, 87.1)
- removed the ? at (59.7, 33.6)
- removed the ? at (63.4, 31.7)
- removed the ? at (43.1, 87.1)
- removed the ? at (57.8, 33.6)
- removed the ? at (63.4, 28.0)
- removed the ? at (64.4, 65.3)
- removed the ? at (61.5, 29.9)
- removed the ? at (57.8, 29.9)
- removed the ? at (61.5, 28.0)
- removed the ? at (61.5, 33.6)
- removed the ? at (57.8, 31.7)
- removed the ? at (57.8, 28.0)
- removed the ? at (65.0, 65.3)
- removed the ? at (63.4, 29.9)
- removed the ? at (59.7, 28.0)
- removed the ? at (59.7, 31.7)
- removed the ? at (44.2, 88.3)
- removed the ? at (63.8, 65.3)
- removed the ? at (59.7, 29.9)
- removed the ? at (61.5, 31.7)
- removed the ? at (43.1, 88.3)
- removed the ? at (63.4, 33.6)
- removed the C15 at (61.3, 64.4)
- removed C16: 104, Capacitor_SMD:C_0805_2012Metric_Pad1.18x1.45mm_HandSolder
- removed C17: 10uF ±10% 10V, My_Personal_Footprints_Library:CL10A106KP8NNNC
- removed C18: 4.7uF, My_Personal_Footprints_Library:CL10A475KP8NNNC
- removed H13: MountingHole, MountingHole:MountingHole_3.2mm_M3
- removed LED2: EMERALD, My_Personal_Footprints_Library:LED_EMERALD_20mA_FC-D1608UGK-520D10
- removed L_B-CH1: 47uH±20% - 680mA, My_Personal_Footprints_Library:ind_47uH_LPS4018-473MRC
- removed the U7 at (40.2, 62.8)
- added ?: , , F.Cu at (126.2, 70.9)
- added ?: , , F.Cu at (124.4, 65.3)
- added ?: , , F.Cu at (128.1, 70.9)
- added ?: , , F.Cu at (126.2, 69.0)
- added ?: , , F.Cu at (122.5, 65.3)
- added ?: , , F.Cu at (122.5, 67.2)
- added ?: , , F.Cu at (126.2, 67.2)
- added ?: , , F.Cu at (122.5, 70.9)
- added ?: , , F.Cu at (124.4, 67.2)
- added ?: , , F.Cu at (128.1, 69.0)
- added ?: , , F.Cu at (124.4, 70.9)
- added ?: , , F.Cu at (129.7, 102.6)
- added ?: , , F.Cu at (128.5, 102.6)
- added ?: , , F.Cu at (128.1, 65.4)
- added ?: , , F.Cu at (124.4, 69.0)
- added ?: , , F.Cu at (126.2, 65.4)
- added ?: , , F.Cu at (122.5, 69.0)
- added ?: , , F.Cu at (128.1, 67.2)
- added ?: , , F.Cu at (129.1, 102.6)
- added Q6: P-MOSFET-ENH-BSS84LT1G, My_Personal_Footprints_Library:BSS84LT1G, F.Cu at (125.7, 114.9)
- added Q7: N-MOSFET-ENH-2N7002, My_Personal_Footprints_Library:2N7002, F.Cu at (132.1, 113.7)
- added SW3: SPDT, My_Personal_Footprints_Library:SS-12F49-G050, F.Cu at (94.5, 94.3)
- added U4: DFR0819, My_Personal_Footprints_Library:DFR0819, F.Cu at (160.6, 97.8)
- C11: value 10uF ±10% 25V -> 10uF ±10% 10V; footprint My_Personal_Footprints_Library:CAP_10uF_CL21A106KAYNNNE -> My_Personal_Footprints_Library:CL10A106KP8NNNC
- C12: value 22nF -> 104; footprint My_Personal_Footprints_Library:CAP_22nF_0402B223K500NT -> Capacitor_SMD:C_0805_2012Metric_Pad1.18x1.45mm_HandSolder
- C13: value 2.2uF ±10% 25V -> 10uF ±10% 10V; footprint My_Personal_Footprints_Library:CAP_2.2uF_GRM155R61E225KE11D -> My_Personal_Footprints_Library:CL10A106KP8NNNC
- C14: value 22uF ±20% 6.3V -> 4.7uF; footprint My_Personal_Footprints_Library:CM05X5R226M06AH080 -> My_Personal_Footprints_Library:CL10A475KP8NNNC
- CARD1: value micro SD Card slot TF PUSH -> micro SD-CARD TF PUSH
- D1, D2, D3: value BAT760-7 -> RB168MM-40TR; footprint Diode_SMD:D_SOD-323F -> My_Personal_Footprints_Library:RB168MM-40TR
- LED1: value RED -> E6C0606RGBC3UDA; footprint My_Personal_Footprints_Library:LED0603-RD_RED -> My_Personal_Footprints_Library:E6C0606RGBC3UDA
- R10: value 10kΩ ±1% 62.5mW -> 150Ω ±1% 62.5mW; footprint My_Personal_Footprints_Library:RES_10K_0402WGF1002TCE -> Resistor_SMD:R_0402_1005Metric
- R11: value 3kΩ ±1% 62.5mW -> 36Ω ±1% 62.5mW; footprint My_Personal_Footprints_Library:FRC04002F3001TS -> Resistor_SMD:R_0402_1005Metric
- R12: value 604Ω -> 36Ω ±1% 62.5mW; footprint My_Personal_Footprints_Library:RTT066040FTP -> Resistor_SMD:R_0402_1005Metric
- R13: value 604Ω -> 10K; footprint My_Personal_Footprints_Library:RTT066040FTP -> Resistor_SMD:R_0805_2012Metric_Pad1.20x1.40mm_HandSolder
- R14: value 1.78MΩ ±1% 62.5mW -> 10K; footprint My_Personal_Footprints_Library:RC0402FR-071M78L -> Resistor_SMD:R_0805_2012Metric_Pad1.20x1.40mm_HandSolder
- R15: value 887kΩ -> 10K; footprint My_Personal_Footprints_Library:RC0402FR-07887KL -> Resistor_SMD:R_0805_2012Metric_Pad1.20x1.40mm_HandSolder
- R16: value 10K -> 100
- R17: value 10K -> 220Ω; footprint Resistor_SMD:R_0805_2012Metric_Pad1.20x1.40mm_HandSolder -> My_Personal_Footprints_Library:0603WAJ0221T5E
- R18: value 10K -> 7.5kΩ; footprint Resistor_SMD:R_0805_2012Metric_Pad1.20x1.40mm_HandSolder -> My_Personal_Footprints_Library:0603WAF7501T5E
- R19: value 100 -> 7.5kΩ; footprint Resistor_SMD:R_0805_2012Metric_Pad1.20x1.40mm_HandSolder -> My_Personal_Footprints_Library:0603WAF7501T5E
- R20: value 220Ω -> 7.5kΩ; footprint My_Personal_Footprints_Library:0603WAJ0221T5E -> My_Personal_Footprints_Library:0603WAF7501T5E
- R24: value 7.5kΩ -> 100; footprint My_Personal_Footprints_Library:0603WAF7501T5E -> Resistor_SMD:R_0805_2012Metric_Pad1.20x1.40mm_HandSolder
- R25: value 7.5kΩ -> 10K; footprint My_Personal_Footprints_Library:0603WAF7501T5E -> Resistor_SMD:R_0805_2012Metric_Pad1.20x1.40mm_HandSolder
- R26: value 7.5kΩ -> 4.7kΩ ±1% 100mW; footprint My_Personal_Footprints_Library:0603WAF7501T5E -> My_Personal_Footprints_Library:0603WAF4701T5E
- SW1: value BOOT -> ~; footprint My_Personal_Footprints_Library:SW_1TS005F-2500-5001 -> My_Personal_Footprints_Library:KMR211NGLFS
- SW2: value RESET -> ~; footprint My_Personal_Footprints_Library:SW_1TS005F-2500-5001 -> My_Personal_Footprints_Library:KMR211NGLFS
- U2: value Screw_Terminal_KF301_1x02 -> ~; footprint My_Personal_Footprints_Library:Screw_Terminal_KF301_1x02 -> My_Personal_Footprints_Library:CONN-TH_S2B-PH-K-S-GW
- moved R19 136.0 mm to (123.2, 137.8), turned to 90 degrees
- moved R18 135.0 mm to (127.7, 137.9)
- moved R17 116.5 mm to (136.5, 101.7), turned to 90 degrees
- moved H5 116.4 mm to (137.2, 148.8), turned to -90 degrees
- moved H8 107.5 mm to (137.2, 136.0), turned to -90 degrees
- moved TP1 107.5 mm to (104.9, 149.9), turned to 0 degrees
- moved C13 102.5 mm to (134.3, 101.8), turned to 90 degrees
- moved H3 102.2 mm to (137.2, 125.9), turned to 90 degrees
- moved H12 102.0 mm to (168.4, 152.3)
- moved CARD1 101.3 mm to (125.3, 147.0), turned to 0 degrees
- moved C14 99.4 mm to (132.1, 101.7), turned to 90 degrees
- moved R21 96.2 mm to (132.3, 135.8), turned to 90 degrees
- moved TP3 95.9 mm to (105.0, 138.9), turned to -90 degrees
- moved C10 93.8 mm to (125.5, 137.2), turned to -90 degrees
- moved H1 91.5 mm to (129.5, 124.7), turned to 90 degrees
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- renumbered C19 to C15, U9 to U6, U10 to U7
Connections:
- C10 pad 2: +3V3 -> /micro_SD-CARD_enable/3V3_Input_to_micro_SD-CARD
- C11 pad 2: EXT_5V -> /Buck-Boost3.3V/Buck-Boost_INPUT
- C12 pad 1: Net-(U7-SW) -> /Buck-Boost3.3V/Buck-Boost_INPUT
- C12 pad 2: Net-(U7-BOOST) -> GND
- C13 pad 1: Net-(U7-INTVcc) -> GND
- C13 pad 2: GND -> +3V3
- C14 pad 2: /Battery_Charger_LiFePO4_3.6V/Battery_Charger_OUTPUT -> +3V3
- CARD1 pad 4: +3V3 -> /micro_SD-CARD_enable/3V3_Input_to_micro_SD-CARD
- D2 pad 1: VBAT -> Net-(D2-C)
- D2 pad 2: /Battery_Charger_LiFePO4_3.6V/Battery_Charger_OUTPUT -> /Battery_Voltage_Monitor_with_MOSFETS/V_Batt_Monitor_INPUT
- H3 pad 2: IO0 -> GND
- H3 pad 3: D4 -> IO0
- H4 pad 3: D27 -> +3V3
- H4 pad 4: D26 -> GND
- H5 pad 4: D21 -> +3V3
- H5 pad 5: D22 -> GND
- H6 pad 2: D33 -> EXT_5V
- LED1 pad 1: Net-(LED1-K) -> Net-(LED1-B)
- LED1 pad 2: Net-(LED1-A) -> +3V3
- Q4 pad 2: /Battery_Charger_LiFePO4_3.6V/Battery_Charger_OUTPUT -> /Battery_Voltage_Monitor_with_MOSFETS/V_Batt_Monitor_INPUT
- R10 pad 1: Net-(U7-MPPT) -> Net-(LED1-R)
- R10 pad 2: EXT_5V -> D33
- R11 pad 1: GND -> D27
- R11 pad 2: Net-(U7-PROG) -> Net-(LED1-B)
- R12 pad 1: Net-(LED1-A) -> D26
- R12 pad 2: EXT_5V -> Net-(LED1-G)
- R13 pad 1: Net-(LED2-A) -> Net-(Q3-D)
- R13 pad 2: EXT_5V -> /Battery_Voltage_Monitor_with_MOSFETS/V_Batt_Monitor_INPUT
- R14 pad 1: Net-(U7-FB) -> D34
- R14 pad 2: Net-(U7-FBG) -> Net-(Q4-D)
- R15 pad 1: /Battery_Charger_LiFePO4_3.6V/Battery_Charger_OUTPUT -> GND
- R15 pad 2: Net-(U7-FB) -> D34
- R16 pad 1: Net-(Q3-D) -> Net-(Q3-G)
- R16 pad 2: /Battery_Charger_LiFePO4_3.6V/Battery_Charger_OUTPUT -> D25
- R17 pad 1: D34 -> GND
- R17 pad 2: Net-(Q4-D) -> +3V3
- R18 pad 1: GND -> D15
- R18 pad 2: D34 -> /micro_SD-CARD_enable/3V3_Input_to_micro_SD-CARD
- R19 pad 1: Net-(Q3-G) -> D14
- R19 pad 2: D25 -> /micro_SD-CARD_enable/3V3_Input_to_micro_SD-CARD
- R20 pad 1: GND -> D2
- R20 pad 2: +3V3 -> /micro_SD-CARD_enable/3V3_Input_to_micro_SD-CARD
- R21 pad 1: D15 -> Net-(CARD1-DAT2)
- R21 pad 2: +3V3 -> /micro_SD-CARD_enable/3V3_Input_to_micro_SD-CARD
- R22 pad 1: D14 -> Net-(CARD1-CD/DAT3)
- R22 pad 2: +3V3 -> /micro_SD-CARD_enable/3V3_Input_to_micro_SD-CARD
- R23 pad 1: D2 -> Net-(CARD1-DAT1)
- R23 pad 2: +3V3 -> /micro_SD-CARD_enable/3V3_Input_to_micro_SD-CARD
- R24 pad 1: Net-(CARD1-DAT2) -> Net-(Q7-G)
- R24 pad 2: +3V3 -> D4
- R25 pad 1: Net-(CARD1-CD/DAT3) -> Net-(Q6-G)
- R26 pad 1: Net-(CARD1-DAT1) -> GND
- R26 pad 2: +3V3 -> /micro_SD-CARD_enable/3V3_Input_to_micro_SD-CARD
- SW1 pad 2: IO0 -> GND
- SW1 pad 3: GND -> IO0
- SW2 pad 2: ENA -> GND
- SW2 pad 3: GND -> ENA
- U2 pad 1: /Battery_Charger_LiFePO4_3.6V/Battery_Charger_OUTPUT -> /Battery_Voltage_Monitor_with_MOSFETS/V_Batt_Monitor_INPUT
Routing:
- net /micro_SD-CARD_enable/3V3_Input_to_micro_SD-CARD: track 0.00 -> 66.9 mm, vias 0 -> 6
- net D33: track 77.8 -> 14.9 mm, vias 1 -> 2
- net /Battery_Charger_LiFePO4_3.6V/Battery_Charger_OUTPUT: track 59.7 -> 0.00 mm
- net EXT_5V: track 164.0 -> 106.1 mm, vias 5 -> 4
- net D23: track 56.0 -> 108.7 mm
- net D19: track 47.5 -> 91.0 mm
- net D26: track 52.8 -> 11.9 mm
- net D18: track 44.2 -> 84.6 mm
- net /Battery_Voltage_Monitor_with_MOSFETS/V_Batt_Monitor_INPUT: track 0.00 -> 38.8 mm, vias 0 -> 1
- net D27: track 47.8 -> 9.57 mm
- net D5: track 40.6 -> 78.0 mm
- net GND: track 150.3 -> 182.0 mm, vias 32 -> 21
- net D2: track 41.8 -> 73.2 mm, vias 1 -> 2
- net IO0: track 120.9 -> 152.0 mm, vias 4 -> 3
- net D15: track 42.5 -> 71.6 mm, vias 0 -> 1
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- removed copper zone on F.Cu, net Net-(U7-CHGSNS)
- removed copper zone on F.Cu, net Net-(U7-SW)
Other:
- board size 97.3 x 90.9 mm -> 87.9 x 98 mm
- board text added: "5V (USB)"
- board text added: "LOW QUIESCENT CURRENT BOARD MODULE: ESP32 WROVER-E WITH 4MB PSRAM SUPPLY: 3.7V LiPO BATTERIES OR 5V USB"
- board text added: "OFF"
- board text added: "ON"
- board text removed: "5V(USB)"
- board text removed: "BATTERY MONITOR (HALF VOLTAGE)"
- board text removed: "BATTERY-CHARGER/SUPPLY LiFePO4 (3.6V OUTPUT)"
- board text removed: "BUTTON SWITCHES"
- board text removed: "ESP32-WROVER-E WITH 4MB PSRAM"
- board text removed: "LOW QUIESCENT CURRENT BOARD MODULE: ESP32 WROVER-E WITH 4MB PSRAM SUPPLY: 3.6V LiFePO4 BATTERIES OR 5V USB"
- board text removed: "PERIPHERALS TEST ZONE"
- board text removed: "USB"

Commit message: Second commit
Parts:
- removed ? (x19): , 
- added C16: 104, Capacitor_SMD:C_0805_2012Metric_Pad1.18x1.45mm_HandSolder, F.Cu at (167.8, 125.4)
- added C17: 104, Capacitor_SMD:C_0805_2012Metric_Pad1.18x1.45mm_HandSolder, F.Cu at (103.1, 98.8)
- added J1: SM04B-SRSS-TB, My_Personal_Footprints_Library:CONN_SM04B-SRSS-TB_JST, F.Cu at (166.3, 133.9)
- added J2: SM04B-SRSS-TB, My_Personal_Footprints_Library:CONN_SM04B-SRSS-TB_JST, F.Cu at (155.1, 133.9)
- added Q10: N-MOSFET-ENH-2N7002, My_Personal_Footprints_Library:2N7002, F.Cu at (170.5, 115.3)
- added Q9: P-MOSFET-ENH-BSS84LT1G, My_Personal_Footprints_Library:BSS84LT1G, F.Cu at (165.6, 121.2)
- added R26: 100, Resistor_SMD:R_0805_2012Metric_Pad1.20x1.40mm_HandSolder, F.Cu at (171.4, 110.8)
- added R28: 4.7kΩ ±1% 100mW, My_Personal_Footprints_Library:0603WAF4701T5E, F.Cu at (167.5, 128.6)
- added R29: 10K, Resistor_SMD:R_0805_2012Metric_Pad1.20x1.40mm_HandSolder, F.Cu at (165.6, 117.9)
- U7: value USB-C_Connector -> USB4110GFA; footprint My_Personal_Footprints_Library:USB3.1C16PFSMT -> My_Personal_Footprints_Library:GCT_USB4110GFA
- moved H10 6.94 mm to (171.3, 58.2)
- moved H9 6.17 mm to (90.7, 58.3)
- moved H12 2.64 mm to (171.1, 152.3)
- moved R3 1.85 mm to (96.4, 132.0)
- moved R4 1.85 mm to (99.1, 132.0)
- moved R5 1.85 mm to (104.4, 132.0)
- moved R6 1.85 mm to (101.7, 132.0)
- moved R7 1.85 mm to (107.0, 132.0)
- moved C5 1.85 mm to (91.1, 132.0)
- moved C9 1.85 mm to (93.8, 132.0)
- moved D1 1.85 mm to (88.6, 132.4)
- moved R1 1.85 mm to (93.3, 138.6)
- moved U7 1.32 mm to (92.3, 120.5)
- moved U4 1.04 mm to (160.6, 96.8)
- moved U6 0.06 mm to (126.3, 72.0)
- renumbered Q6 to Q8, R26 to R27
Connections:
- H5 pad 1: D5 -> GND
Routing:
- net D21: track 34.9 -> 114.1 mm, vias 2 -> 5
- net D22: track 39.4 -> 109.6 mm, vias 2 -> 5
- net +3V3: track 305.8 -> 363.4 mm, vias 10 -> 13
- net GND: track 182.0 -> 226.4 mm, vias 21 -> 32
- net D5: track 78.0 -> 64.4 mm, vias 1 -> 4
- net /I2C_Connector_Enable/3V3_Input_to_I2C_Connector: track 0.00 -> 9.95 mm
- net Net-(Q10-D): track 0.00 -> 6.83 mm
- net VBAT: track 12.7 -> 18.1 mm
- net Net-(Q10-G): track 0.00 -> 2.58 mm
- net Net-(U3-VBUS): track 10.6 -> 12.4 mm
- net Net-(U3-~{RST}): track 6.91 -> 8.78 mm
- net Net-(U3-~{SUSPEND}): track 7.15 -> 8.98 mm
- net VBUS: track 39.0 -> 40.6 mm
- net EXT_5V: track 106.1 -> 105.2 mm
Other:
- board size 87.9 x 98 mm -> 90.5 x 104.2 mm
- board text added: "LOW QUIESCENT CURRENT BOARD MODULE: ESP32 WROVER-E-N4R8 SUPPLY: BATTERIES OR 5V USB DATE: 06/2025 V1.0 G.L."
- board text added: "LiPO 3.7V"
- board text removed: "LOW QUIESCENT CURRENT BOARD MODULE: ESP32 WROVER-E WITH 4MB PSRAM SUPPLY: 3.7V LiPO BATTERIES OR 5V USB"
- board text removed: "USB-SERIAL"

Commit message: Third commit
Other:
- board text added: "EXT5V"
- board text added: "I2C CONNECTORS"
- board text removed: "D21"
- board text removed: "D22"
- board text removed: "D26"
- board text removed: "D27"
- board text removed: "D33"
- board text removed: "D4"
- board text removed: "D5"

Commit message: Fourth commit
Parts:
- R10, R11, R12: footprint Resistor_SMD:R_0402_1005Metric -> My_Personal_Footprints_Library:RES_10K_0402WGF1002TCE
- moved Q5 0.11 mm to (105.0, 94.1)
- moved U2 0.09 mm to (92.3, 108.8)
- moved Q3 0.08 mm to (97.0, 78.7)
- moved D1 0.07 mm to (88.6, 132.5)
- moved U6 0.07 mm to (126.3, 72.0)
- moved Q10 0.07 mm to (170.5, 115.2)
- moved D2 0.06 mm to (89.8, 94.5)
Routing:
- net GND: track 226.4 -> 267.7 mm, vias 32 -> 31
- net +3V3: track 363.4 -> 384.1 mm, vias 13 -> 12
- net /Buck-Boost3.3V/Buck-Boost_INPUT: track 43.3 -> 55.5 mm
- net Net-(U5-L2): track 0.79 -> 10.3 mm
- net Net-(U5-L1): track 0.81 -> 10.1 mm
- net VBUS: track 40.6 -> 46.1 mm
- net VBAT: track 18.1 -> 15.2 mm
- net DTR: track 13.9 -> 11.5 mm
- net D14: track 74.0 -> 71.9 mm
- net D15: track 71.6 -> 69.9 mm
- net D2: track 73.2 -> 71.5 mm
- net EXT_5V: track 105.2 -> 104.2 mm
- net Net-(D2-C): track 6.31 -> 5.28 mm
- net D12: track 64.7 -> 63.8 mm
- net IO0: track 152.0 -> 151.1 mm
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Other:
- rule pad_to_mask_clearance: 0 -> 0.1

Commit message: 5th commit
Parts:
- removed H3, H4: Header-Female-2.54_1x4, My_Personal_Footprints_Library:Header-Female-2.54_1x4
- added C18: 104, Capacitor_SMD:C_0805_2012Metric_Pad1.18x1.45mm_HandSolder, F.Cu at (129.5, 106.9)
- added Q11: P-MOSFET-ENH-BSS84LT1G, My_Personal_Footprints_Library:BSS84LT1G, F.Cu at (123.8, 103.8)
- added Q12: N-MOSFET-ENH-2N7002, My_Personal_Footprints_Library:2N7002, F.Cu at (124.9, 96.6)
- added R30: 4.7kΩ ±1% 100mW, My_Personal_Footprints_Library:0603WAF4701T5E, F.Cu at (126.9, 106.6)
- added R31: 100, Resistor_SMD:R_0805_2012Metric_Pad1.20x1.40mm_HandSolder, F.Cu at (129.2, 95.6)
- added R32: 10K, Resistor_SMD:R_0805_2012Metric_Pad1.20x1.40mm_HandSolder, F.Cu at (123.9, 99.9)
- added REF**: BEE_LOGO, My_Personal_Footprints_Library:BEE_LOGO, F.Cu at (169.4, 52.5)
- moved H6 46.2 mm to (158.0, 133.8), turned to 0 degrees
- moved H8 32.3 mm to (169.4, 133.8), turned to 0 degrees
- moved TP1 23.6 mm to (104.7, 126.2)
- moved C10 23.3 mm to (139.6, 118.7)
- moved CARD1 23.3 mm to (139.4, 128.5)
- moved H1 23.3 mm to (143.6, 106.1)
- moved H2 23.3 mm to (136.0, 106.1)
- moved Q8 23.3 mm to (139.8, 96.4)
- moved R18 23.3 mm to (141.7, 119.3)
- moved R21 23.3 mm to (146.3, 117.2)
- moved R23 23.3 mm to (132.3, 119.8)
- moved Q7 23.3 mm to (146.1, 95.1)
- moved R19 23.3 mm to (137.2, 119.2)
- moved R22 23.3 mm to (144.3, 117.4)
- moved R24 23.3 mm to (150.4, 96.1)
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Connections:
- H1 pad 3: D2 -> D14
- H2 pad 2: +3V3 -> 3V3_ON_OFF
- H2 pad 3: D13 -> D2
- H5 pad 2: D18 -> 3V3_ON_OFF
- H5 pad 3: D19 -> D13
- H5 pad 4: +3V3 -> D32
- H5 pad 5: GND -> D35
- H5 pad 6: D23 -> GND
- H6 pad 2: EXT_5V -> +3V3
- H6 pad 3: D32 -> IO0
- H6 pad 4: D35 -> D19
- H6 pad 5: GND -> D23
- H7 pad 1: EXT_5V -> GND
- H7 pad 2: GND -> EXT_5V
- H8 pad 1: +3V3 -> SENSOR_VN
- H8 pad 2: GND -> SENSOR_VP
- U6 pad 4: unconnected-(U6-SENSOR_VP-Pad4) -> SENSOR_VP
- U6 pad 5: unconnected-(U6-SENSOR_VN-Pad5) -> SENSOR_VN
Routing:
- net SENSOR_VP: track 0.00 -> 151.9 mm, vias 0 -> 1
- net SENSOR_VN: track 0.00 -> 127.3 mm, vias 0 -> 1
- net 3V3_ON_OFF: track 0.00 -> 47.9 mm, vias 0 -> 1
- net IO0: track 151.1 -> 181.2 mm
- net D18: track 83.8 -> 55.5 mm, vias 1 -> 2
- net +3V3: track 384.1 -> 359.6 mm, vias 12 -> 13
- net D13: track 55.5 -> 77.3 mm
- net GND: track 267.7 -> 282.4 mm, vias 31 -> 34
- net D14: track 71.9 -> 82.3 mm, vias 2 -> 1
- net EXT_5V: track 104.2 -> 93.9 mm
- net D32: track 80.8 -> 88.8 mm
- net Net-(Q11-G): track 0.00 -> 5.09 mm
- net D4: track 44.8 -> 49.8 mm
- net D2: track 71.5 -> 76.1 mm
- net D23: track 107.9 -> 103.4 mm
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Other:
- board text added: "5V"
- board text added: "VN"
- board text added: "VP"
- board text removed: "D18"
- board text removed: "EXT5V"

Commit message: 5th commit
Parts:
- moved H8 85.1 mm to (180.9, 49.5), turned to 90 degrees
- moved H6 4.32 mm to (153.7, 133.8)
- moved CARD1 3.48 mm to (135.9, 128.5)
- moved R21 3.48 mm to (142.9, 117.2)
- moved R23 3.48 mm to (128.8, 119.8)
- moved C10 3.48 mm to (136.1, 118.7)
- moved R18 3.48 mm to (138.2, 119.3)
- moved R19 3.48 mm to (133.8, 119.2)
- moved R20 3.48 mm to (131.5, 120.1)
- moved R22 3.48 mm to (140.8, 117.4)
- moved H5 2.50 mm to (118.0, 133.8)
- moved H7 2.50 mm to (106.6, 133.8)
Routing:
- net SENSOR_VP: track 151.9 -> 57.9 mm
- net SENSOR_VN: track 127.3 -> 58.3 mm
- net D14: track 82.3 -> 85.8 mm
- net D15: track 71.6 -> 74.6 mm
- net +3V3: track 359.6 -> 361.4 mm
- net D23: track 103.4 -> 101.6 mm
- net IO0: track 181.2 -> 179.4 mm
- net D19: track 93.4 -> 91.6 mm
- net D2: track 76.1 -> 77.6 mm
- net /micro_SD-CARD_enable/3V3_Input_to_micro_SD-CARD: track 68.6 -> 67.1 mm
- net EXT_5V: track 93.9 -> 95.0 mm
- net D32: track 88.8 -> 89.9 mm
- net D35: track 88.5 -> 89.5 mm
- net D13: track 77.3 -> 78.4 mm
- net 3V3_ON_OFF: track 47.9 -> 49.0 mm
