File: Kicad9_projects_folder/MY-ESP32/MY-ESP32.kicad_pcb (KiCad board)
At the start: 4 copper layers, 90.5 x 104.2 mm, 95 parts, among them J1 SM04B-SRSS-TB, J2 SM04B-SRSS-TB, Q1 2N3904S-RTK/PS, Q10 N-MOSFET-ENH-2N7002, Q11 P-MOSFET-ENH-BSS84LT1G, Q12 N-MOSFET-ENH-2N7002, Q2 2N3904S-RTK/PS, Q3 N-MOSFET-ENH-2N7002, Q4 P-MOSFET-ENH-BSS84LT1G, Q5 PMOSFET-DMP1045U-7, Q7 N-MOSFET-ENH-2N7002, Q8 P-MOSFET-ENH-BSS84LT1G, Q9 P-MOSFET-ENH-BSS84LT1G, SW3 SPDT, U1 USBLC6-2SC6, U3 CP2102N-Axx-xQFN28, U4 DFR0819, U5 TPS63001DRCR, U7 USB4110GFA

Commit message: 5th commit
Parts:
- removed the H8 at (180.9, 49.5)
- removed REF**: BEE_LOGO, My_Personal_Footprints_Library:BEE_LOGO
- added H6: Header-Female-2.54_1x2, My_Personal_Footprints_Library:Header-Female-2.54_1x2, F.Cu at (180.9, 49.5)
- renumbered H12 to H10, H5 to H3, H6 to H4, H7 to H5, H9 to H7, H10 to H8, H11 to H9, Q11 to Q10, Q12 to Q11, Q7 to Q6, Q8 to Q7, Q9 to Q8, Q10 to Q9

Commit message: 6th commit
Parts:
- removed LED1: E6C0606RGBC3UDA, My_Personal_Footprints_Library:E6C0606RGBC3UDA
- removed R10: 150Ω ±1% 62.5mW, My_Personal_Footprints_Library:RES_10K_0402WGF1002TCE
- removed R11, R12: 36Ω ±1% 62.5mW, My_Personal_Footprints_Library:RES_10K_0402WGF1002TCE
- added LED2: E6C0606RGBC3UDA, My_Personal_Footprints_Library:E6C0606RGBC3UDA, F.Cu at (120.8, 66.9)
- added R33: 36Ω ±1% 62.5mW, My_Personal_Footprints_Library:RES_10K_0402WGF1002TCE, F.Cu at (121.2, 62.8)
- added R34: 36Ω ±1% 62.5mW, My_Personal_Footprints_Library:RES_10K_0402WGF1002TCE, F.Cu at (122.8, 62.8)
- added R35: 150Ω ±1% 62.5mW, My_Personal_Footprints_Library:RES_10K_0402WGF1002TCE, F.Cu at (119.6, 62.8)
Routing:
- net +3V3: track 361.4 -> 314.2 mm, vias 13 -> 12
- net 3V3_ON_OFF: track 49.0 -> 92.7 mm, vias 1 -> 3
- net Net-(LED2-R): track 0.00 -> 5.50 mm
- net Net-(LED1-R): track 5.50 -> 0.00 mm
- net Net-(LED2-B): track 0.00 -> 3.61 mm
- net Net-(LED1-B): track 3.61 -> 0.00 mm
- net Net-(LED2-G): track 0.00 -> 3.32 mm
- net Net-(LED1-G): track 3.32 -> 0.00 mm
- net D18: track 55.5 -> 57.7 mm

Commit message: 6th commit
Parts:
- removed LED2: E6C0606RGBC3UDA, My_Personal_Footprints_Library:E6C0606RGBC3UDA
- added LED1: TJ-S1615CY6TGLCCSRGB-A5, My_Personal_Footprints_Library:TJ-S1615CY6TGLCCSRGB-A5, F.Cu at (121.2, 67.4)
- moved R34 0.06 mm to (122.9, 62.8), turned to 90 degrees
- turned R33 to 90 degrees
Connections:
- R33 pad 1: D26 -> Net-(LED1-G)
- R33 pad 2: Net-(LED2-G) -> D26
- R34 pad 1: D27 -> Net-(LED1-B)
- R34 pad 2: Net-(LED2-B) -> D27
Routing:
- net 3V3_ON_OFF: track 92.7 -> 49.0 mm, vias 3 -> 1
- net Net-(LED1-B): track 0.00 -> 6.10 mm
- net Net-(LED1-G): track 0.00 -> 4.03 mm
- net Net-(LED2-B): track 3.61 -> 0.00 mm
- net Net-(LED2-G): track 3.32 -> 0.00 mm
- net GND: track 282.4 -> 284.5 mm, vias 34 -> 35
- net Net-(LED1-R): track 5.50 -> 4.16 mm
