File: Kicad9_projects_folder/MY-ESP32/3V3_Headers_enable.kicad_sch (KiCad schematic)
At the start: 5 parts, among them Q11 P-MOSFET-ENH-BSS84LT1G, Q12 N-MOSFET-ENH-2N7002

Commit message: 5th commit
Parts:
- renumbered Q11 to Q10, Q12 to Q11
Changed lines of the file:
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@@
 		(dnp no)
 		(fields_autoplaced yes)
-		(property "Reference" "Q12"
+		(property "Reference" "Q11"
 			(at 198.12 113.0299 0)
 			(effects
@@
 			(project "MY-ESP32"
 				(path "/d6d8d651-8dd4-45a4-bd17-f84a87bbb30c/b3780aea-0409-4b0e-9d6e-ab9fc89bcb41"
-					(reference "Q12")
+					(reference "Q11")
 					(unit 1)
 				)
@@
 		(dnp no)
 		(fields_autoplaced yes)
-		(property "Reference" "Q11"
+		(property "Reference" "Q10"
 			(at 96.52 72.3899 0)
 			(effects
@@
 			(project "MY-ESP32"
 				(path "/d6d8d651-8dd4-45a4-bd17-f84a87bbb30c/b3780aea-0409-4b0e-9d6e-ab9fc89bcb41"
-					(reference "Q11")
+					(reference "Q10")
 					(unit 1)
 				)
