File: Kicad9_projects_folder/MY-ESP32/I2C_Connector_Enable.kicad_sch (KiCad schematic)
At the start: 5 parts, among them Q10 N-MOSFET-ENH-2N7002, Q9 P-MOSFET-ENH-BSS84LT1G

Commit message: 5th commit
Parts:
- renumbered Q9 to Q8, Q10 to Q9
Changed lines of the file:
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@@
 		(dnp no)
 		(fields_autoplaced yes)
-		(property "Reference" "Q10"
+		(property "Reference" "Q9"
 			(at 200.66 107.9499 0)
 			(effects
@@
 			(project "MY-ESP32"
 				(path "/d6d8d651-8dd4-45a4-bd17-f84a87bbb30c/6919b8a3-84d4-45ca-a14c-74be4024a5b9"
-					(reference "Q10")
+					(reference "Q9")
 					(unit 1)
 				)
@@
 		(dnp no)
 		(fields_autoplaced yes)
-		(property "Reference" "Q9"
+		(property "Reference" "Q8"
 			(at 99.06 67.3099 0)
 			(effects
@@
 			(project "MY-ESP32"
 				(path "/d6d8d651-8dd4-45a4-bd17-f84a87bbb30c/6919b8a3-84d4-45ca-a14c-74be4024a5b9"
-					(reference "Q9")
+					(reference "Q8")
 					(unit 1)
 				)
