File: Kicad9_projects_folder/MY-ESP32/MY-ESP32.kicad_sch (KiCad schematic)
At the start: 56 parts, among them Q1 2N3904S-RTK/PS, Q2 2N3904S-RTK/PS, Q5 PMOSFET-DMP1045U-7, SW1 BOOT, SW2 RESET, U1 USBLC6-2SC6, U10 USB-C_Connector, U11 TPS3839G33DBZR, U2 Screw_Terminal_KF301_1x02, U3 CP2102N-Axx-xQFN28

Commit message: Second commit
Parts:
- added R24, R25, R26: 7.5kΩ, My_Personal_Footprints_Library:0603WAF7501T5E, symbol My_Personal_Symbols_Library:0603WAF7501T5E
Connections:
- net +3V3: now also R24.2, R25.2, R26.2
- net at CARD1.1 (DAT2): now also R24.1
- net at CARD1.2 (CD/DAT3): now also R25.1
- net at CARD1.8 (DAT1): now also R26.1
- no-connect marks 34 -> 31
Other:
- moved on the sheet: C10, CARD1, R21, R22, R23, TP1

Commit message: Third commit
Parts:
- removed U11: TPS3839G33DBZR, My_Personal_Footprints_Library:TPS3839G33DBZR, symbol My_Personal_Symbols_Library:TPS3839G33DBZR
Other:
- sheet Buck-Boost3.3V ports: added none; removed Buck-Boost_EN
- note removed: "The TPS3839G33 is a voltage supervisor that takes in input the voltage coming from the USB-C or from the batteries. If this voltage (VDD) is over the threshold of 3.08 Volts (VTH) at a given time tx, then, after 200ms (tx+200ms), if VDD is over VTH, it gives in output (RESET#) an high signal (of about VDD-0.4V), otherwise, it stays low. Anyway, if at any moment the VDD signal goes below VTH, the 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"

Commit message: Second commit
Parts:
- removed D1, D2, D3: BAT760-7, Diode_SMD:D_SOD-323F, symbol Device:D_Schottky
- removed H13: MountingHole, MountingHole:MountingHole_3.2mm_M3, symbol Mechanical:MountingHole
- removed SW1: BOOT, My_Personal_Footprints_Library:SW_1TS005F-2500-5001, symbol My_Personal_Symbols_Library:1TS005F-2500-5001
- removed SW2: RESET, My_Personal_Footprints_Library:SW_1TS005F-2500-5001, symbol My_Personal_Symbols_Library:1TS005F-2500-5001
- removed U2: Screw_Terminal_KF301_1x02, My_Personal_Footprints_Library:Screw_Terminal_KF301_1x02, symbol My_Personal_Symbols_Library:KF301-5.0-2P
- added D1, D2, D3: RB168MM-40TR, My_Personal_Footprints_Library:RB168MM-40TR, symbol My_Personal_Symbols_Library:RB168MM-40TR
- added LED1: E6C0606RGBC3UDA, My_Personal_Footprints_Library:E6C0606RGBC3UDA, symbol My_Personal_Symbols_Library:E6C0606RGBC3UDA
- added R10: 150Ω ±1% 62.5mW, Resistor_SMD:R_0402_1005Metric, symbol My_Personal_Symbols_Library:0402WGF1002TCE
- added R11, R12: 36Ω ±1% 62.5mW, Resistor_SMD:R_0402_1005Metric, symbol My_Personal_Symbols_Library:0402WGF1002TCE
- added SW1, SW2: ~, My_Personal_Footprints_Library:KMR211NGLFS, symbol My_Personal_Symbols_Library:KMR211NGLFS
- added SW3: SPDT, My_Personal_Footprints_Library:SS-12F49-G050, symbol My_Personal_Symbols_Library:SS-12F49-G050
- added U2: ~, My_Personal_Footprints_Library:CONN-TH_S2B-PH-K-S-GW, symbol My_Personal_Symbols_Library:S2B-PH-K-S-GW
- added U4: DFR0819, My_Personal_Footprints_Library:DFR0819, symbol My_Personal_Symbols_Library:DFR0819
- CARD1: value micro SD Card slot TF PUSH -> micro SD-CARD TF PUSH
- renumbered C19 to C15, R21 to R18, R22 to R19, R23 to R20, R24 to R21, R25 to R22, R26 to R23, U9 to U6, U10 to U7
Connections:
- net +3V3: now also H4.3, H5.4, LED1.2 (+), U4.1 (VCC); no longer C10.2, CARD1.4 (VDD), R18.2, R19.2, R20.2, R21.2, R22.2, R23.2
- net Buck-Boost3.3V/Buck-Boost_INPUT: now also D3.1 (C)
- net D21: now also U4.4 (SDA); no longer H5.4
- net D22: now also U4.3 (SCL); no longer H5.5
- net D26: now also R12.1; no longer H4.4
- net D27: now also R11.1; no longer H4.3
- net D33: now also R10.2; no longer H6.2
- net D4: no longer H3.3
- net ENA: now also SW2.1, SW2.3
- net EXT_5V: now also H6.2, D1.1 (C), D3.2 (A)
- net GND: now also H3.2, H4.4, H5.5, SW1.2, SW1.4, SW2.2, SW2.4, SW3.4, SW3.5, U2.2, U4.2 (GND)
- net IO0: now also H3.3, SW1.1, SW1.3; no longer H3.2
- net VBAT: now also SW3.1
- net VBUS: now also D1.2 (A)
- new net: D2.1 (C), SW3.2
- new net: LED1.4 (R), R10.1
- new net: LED1.1 (B), R11.2
- new net: LED1.3 (G), R12.2
- new net Battery_Voltage_Monitor_with_MOSFETS/V_Batt_Monitor_INPUT: D2.2 (A), U2.1
- new net micro_SD-CARD_enable/3V3_Input_to_micro_SD-CARD: C10.2, CARD1.4 (VDD), R18.2, R19.2, R20.2, R21.2, R22.2, R23.2
- no-connect marks 31 -> 35
Other:
- removed sheet Battery_Charger_LiFePO4_3.6V
- added sheet micro_SD-CARD_enable (micro_SD-CARD_enable.kicad_sch)
- note added: "BOOT"
- note added: "D21: per SDA del RTC DFR0819"
- note added: "D22: per SCL del RTC DFR0819"
- note added: "D26: dedicato al colore GREEN del led RGB"
- note added: "D27: dedicato al colore BLUE del led RGB"
- note added: "D33: dedicato al colore RED del led RGB"
- note added: "D4: per controllare l'NMOS che connette la micro SD-CARD"
- note added: "LED RGB"
- note added: "MOUNTING HOLES"
- note added: "RESET"
- note added: "RTC"
- note added: "SPDT(Single Pole Double Throw) When the battery is connected to the circuit, then if: -the switch is toggled towards 1 --> 2 shorts with 1 (connection to circuit)--> the circuit can be powered by the battery. -the switch is toggled towards 3 --> 2 shorts with 3 (floating) --> the circuit cannot be powered by the battery."
- moved on the sheet: C1, C10, C15, C2, C3, C4, C5, C6, C7, C8, C9, H1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

Commit message: Second commit
Parts:
- removed U7: USB-C_Connector, My_Personal_Footprints_Library:USB3.1C16PFSMT, symbol My_Personal_Symbols_Library:USB3.1C16PFSMT
- added C16, C17: 104, Capacitor_SMD:C_0805_2012Metric_Pad1.18x1.45mm_HandSolder, symbol Device:C
- added J1, J2: SM04B-SRSS-TB, My_Personal_Footprints_Library:CONN_SM04B-SRSS-TB_JST, symbol My_Personal_Symbols_Library:SM04B-SRSS-TB
- added U7: USB4110GFA, My_Personal_Footprints_Library:GCT_USB4110GFA, symbol My_Personal_Symbols_Library:USB4110GFA
Connections:
- net +3V3: now also J2.3 (3V3)
- net D21: now also J1.2 (SDA), J2.2 (SDA)
- net D22: now also J1.1 (SCL), J2.1 (SCL)
- net D5: no longer H5.1
- net DN: now also U7.A7 (DN1), U7.B7 (DN2)
- net DP: now also U7.A6 (DP1), U7.B6 (DP2)
- net GND: now also H5.1, C16.1, C17.1, J1.4 (GND), J1.5, J1.6, J2.4 (GND), J2.5, J2.6, U7.A1/B12 (GND), U7.B1/A12 (GND), U7.S1 (GND), U7.S2 (GND), U7.S3 (GND), U7.S4 (GND)
- net VBAT: now also C17.2
- net VBUS: now also U7.A4/B9 (VBUS), U7.B4/A9 (VBUS)
- new net I2C_Connector_Enable/3V3_Input_to_I2C_Connector: C16.2, J1.3 (3V3)
Other:
- added sheet I2C_Connector_Enable (I2C_Connector_Enable.kicad_sch)
- note added: "D5: per controllare l'NMOS che connette un connettore I2C"

Commit message: Fourth commit
Parts:
- R10, R11, R12: footprint Resistor_SMD:R_0402_1005Metric -> My_Personal_Footprints_Library:RES_10K_0402WGF1002TCE
Other:
- note added: "I2C"
- moved on the sheet: C16, J1, J2, U4

Commit message: 5th commit
Parts:
- removed H3, H4: Header-Female-2.54_1x4, My_Personal_Footprints_Library:Header-Female-2.54_1x4, symbol My_Personal_Symbols_Library:Header-Female-2.54_1x4
- added C18: 104, Capacitor_SMD:C_0805_2012Metric_Pad1.18x1.45mm_HandSolder, symbol Device:C
Connections:
- net +3V3: now also H6.2; no longer H2.2, H5.4, H8.1
- net D13: now also H5.3; no longer H2.3
- net D14: now also H1.3
- net D18: no longer H5.2
- net D19: now also H6.4; no longer H5.3
- net D2: now also H2.3; no longer H1.3
- net D23: now also H6.5; no longer H5.6
- net D32: now also H5.4; no longer H6.3
- net D35: now also H5.5; no longer H6.4
- net EXT_5V: now also H7.2; no longer H6.2, H7.1
- net GND: now also H5.6, H7.1, C18.1; no longer H5.5, H6.5, H7.2, H8.2
- net IO0: now also H6.3
- net SENSOR_VP: now reaches U6.4 (SENSOR_VP)
- net SENSOR_VP: now also H8.2
- net SENSOR_VN: now reaches U6.5 (SENSOR_VN)
- net SENSOR_VN: now also H8.1
- new net 3V3_ON_OFF: C18.2, H2.2, H5.2
- no-connect marks 35 -> 33
Other:
- added sheet 3V3_Headers_enable (3V3_Headers_enable.kicad_sch)
- note added: "D2: per SD_MMC_D0 e I2S_SD"
- note removed: "D13: per I2S_SD"
- note removed: "D2: per SD_MMC_D0 e I2S_SCK"
- note removed: "GND: per il GND del mic"
- moved on the sheet: H1, H2, H5, H6, LED1, R10, R11, R12

Commit message: 5th commit
Parts:
- renumbered H12 to H10, H5 to H3, H6 to H4, H7 to H5, H8 to H6, H9 to H7, H10 to H8, H11 to H9
Changed lines of the file:
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@@
 		(dnp no)
 		(fields_autoplaced yes)
-		(property "Reference" "H6"
-			(at 483.87 182.2449 0)
+		(property "Reference" "H4"
+			(at 483.87 181.6099 0)
 			(effects
 				(font
@@
 		)
 		(property "Value" "Header-Female-2.54_1x6"
-			(at 483.87 184.15 0)
+			(at 483.87 184.1499 0)
 			(effects
 				(font
@@
 			(project "MY-ESP32"
 				(path "/d6d8d651-8dd4-45a4-bd17-f84a87bbb30c"
-					(reference "H6")
+					(reference "H4")
 					(unit 1)
 				)
@@
 		(dnp no)
 		(fields_autoplaced yes)
-		(property "Reference" "H7"
-			(at 415.29 201.2949 0)
+		(property "Reference" "H5"
+			(at 415.29 200.6599 0)
 			(effects
 				(font
@@
 		)
 		(property "Value" "Header-Female-2.54_1x2"
-			(at 415.29 203.2 0)
+			(at 415.29 203.1999 0)
 			(effects
 				(font
@@
 			(project ""
 				(path "/d6d8d651-8dd4-45a4-bd17-f84a87bbb30c"
-					(reference "H7")
+					(reference "H5")
 					(unit 1)
 				)
@@
 		(dnp no)
 		(fields_autoplaced yes)
-		(property "Reference" "H12"
+		(property "Reference" "H10"
 			(at 38.1 387.3499 0)
 			(effects
@@
 			(project "MY-ESP32"
 				(path "/d6d8d651-8dd4-45a4-bd17-f84a87bbb30c"
-					(reference "H12")
+					(reference "H10")
 					(unit 1)
 				)
@@
 		(dnp no)
 		(fields_autoplaced yes)
-		(property "Reference" "H5"
-			(at 415.29 182.2449 0)
+		(property "Reference" "H3"
+			(at 415.29 181.6099 0)
 			(effects
 				(font
@@
 		)
 		(property "Value" "Header-Female-2.54_1x6"
-			(at 415.29 184.15 0)
+			(at 415.29 184.1499 0)
 			(effects
 				(font
@@
 			(project ""
 				(path "/d6d8d651-8dd4-45a4-bd17-f84a87bbb30c"
-					(reference "H5")
+					(reference "H3")
 					(unit 1)
 				)
@@
 		(dnp no)
 		(fields_autoplaced yes)
-		(property "Reference" "H9"
+		(property "Reference" "H7"
 			(at 38.1 360.6799 0)
 			(effects
@@
 			(project "MY-ESP32"
 				(path "/d6d8d651-8dd4-45a4-bd17-f84a87bbb30c"
-					(reference "H9")
+					(reference "H7")
 					(unit 1)
 				)
@@
 		(dnp no)
 		(fields_autoplaced yes)
-		(property "Reference" "H10"
+		(property "Reference" "H8"
 			(at 38.1 369.5699 0)
 			(effects
@@
 			(project "MY-ESP32"
 				(path "/d6d8d651-8dd4-45a4-bd17-f84a87bbb30c"
-					(reference "H10")
+					(reference "H8")
 					(unit 1)
 				)
@@
 		(dnp no)
 		(fields_autoplaced yes)
-		(property "Reference" "H8"
-			(at 483.87 201.2949 0)
+		(property "Reference" "H6"
+			(at 483.87 200.6599 0)
 			(effects
 				(font
@@
 		)
 		(property "Value" "Header-Female-2.54_1x2"
-			(at 483.87 203.2 0)
+			(at 483.87 203.1999 0)
 			(effects
 				(font
@@
 			(project ""
 				(path "/d6d8d651-8dd4-45a4-bd17-f84a87bbb30c"
-					(reference "H8")
+					(reference "H6")
 					(unit 1)
 				)
@@
 		(dnp no)
 		(fields_autoplaced yes)
-		(property "Reference" "H11"
+		(property "Reference" "H9"
 			(at 38.1 378.4599 0)
 			(effects
@@
 			(project "MY-ESP32"
 				(path "/d6d8d651-8dd4-45a4-bd17-f84a87bbb30c"
-					(reference "H11")
+					(reference "H9")
 					(unit 1)
 				)
