File: Kicad9_projects_folder/MY-ESP32/MY-ESP32.kicad_sch (KiCad schematic)
At the start: 66 parts, among them J1 SM04B-SRSS-TB, J2 SM04B-SRSS-TB, Q1 2N3904S-RTK/PS, Q2 2N3904S-RTK/PS, Q5 PMOSFET-DMP1045U-7, SW3 SPDT, U1 USBLC6-2SC6, U3 CP2102N-Axx-xQFN28, U4 DFR0819, U7 USB4110GFA

Commit message: 6th commit
Parts:
- removed LED2: E6C0606RGBC3UDA, My_Personal_Footprints_Library:E6C0606RGBC3UDA, symbol My_Personal_Symbols_Library:E6C0606RGBC3UDA
- added LED1: TJ-S1615CY6TGLCCSRGB-A5, My_Personal_Footprints_Library:TJ-S1615CY6TGLCCSRGB-A5, symbol My_Personal_Symbols_Library:TJ-S1615CY6TGLCCSRGB-A5
Connections:
- net D26: now also R33.2; no longer R33.1
- net D27: now also R34.2; no longer R34.1
- net GND: now also LED1.1 (C)
- net at R35.1: now also LED1.4 (R)
- new net: LED1.3 (G), R33.1
- new net: LED1.2 (B), R34.1
Other:
- moved on the sheet: R33, R35
