File: Kicad9_projects_folder/MY-ESP32/micro_SD-CARD_enable.kicad_sch (KiCad schematic)
At the start: 5 parts, among them Q6 P-MOSFET-ENH-BSS84LT1G, Q7 N-MOSFET-ENH-2N7002

Commit message: Second commit
Parts:
- renumbered Q6 to Q8, R26 to R27
Changed lines of the file:
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@@
 		(on_board yes)
 		(dnp no)
-		(property "Reference" "R26"
+		(property "Reference" "R27"
 			(at 102.87 120.6499 90)
 			(effects
@@
 			(project ""
 				(path "/d6d8d651-8dd4-45a4-bd17-f84a87bbb30c/b05cfee3-cdbd-4ba0-a586-ca5aad6ef209"
-					(reference "R26")
+					(reference "R27")
 					(unit 1)
 				)
@@
 		(dnp no)
 		(fields_autoplaced yes)
-		(property "Reference" "Q6"
+		(property "Reference" "Q8"
 			(at 95.25 68.5799 0)
 			(effects
@@
 			(project ""
 				(path "/d6d8d651-8dd4-45a4-bd17-f84a87bbb30c/b05cfee3-cdbd-4ba0-a586-ca5aad6ef209"
-					(reference "Q6")
+					(reference "Q8")
 					(unit 1)
 				)

Commit message: 5th commit
Parts:
- renumbered Q7 to Q6, Q8 to Q7
Changed lines of the file:
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@@
 		(dnp no)
 		(fields_autoplaced yes)
-		(property "Reference" "Q7"
+		(property "Reference" "Q6"
 			(at 196.85 109.2199 0)
 			(effects
@@
 			(project "MY-ESP32"
 				(path "/d6d8d651-8dd4-45a4-bd17-f84a87bbb30c/b05cfee3-cdbd-4ba0-a586-ca5aad6ef209"
-					(reference "Q7")
+					(reference "Q6")
 					(unit 1)
 				)
@@
 		(dnp no)
 		(fields_autoplaced yes)
-		(property "Reference" "Q8"
+		(property "Reference" "Q7"
 			(at 95.25 68.5799 0)
 			(effects
@@
 			(project ""
 				(path "/d6d8d651-8dd4-45a4-bd17-f84a87bbb30c/b05cfee3-cdbd-4ba0-a586-ca5aad6ef209"
-					(reference "Q8")
+					(reference "Q7")
 					(unit 1)
 				)
